File: Hardware/SHY.brd (EAGLE design)
At the start: 160 x 100 mm, 14 parts

Commit message: add few components
Parts:
- added U$1: LSM6DS3_CAST, LinnesLab-Sensors:LSM6DS3_CAST
- added U1: (no value), LinnesLab-Microcontrollers:ARTEMIS_CAST
Connections:
- new net SCL: U$1.3
- new net SDA: U$1.4
- net GND: now also U$1.1
Changed lines of the file:
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@@
 <attribute name="VALUE" x="9.5504" y="14.1478" size="1.27" layer="27"/>
+</element>
+<element name="U$1" library="LinnesLab-Sensors" package="LSM6DS3_CAST" value="LSM6DS3_CAST" x="-3.81" y="5.08" smashed="yes">
+<attribute name="NAME" x="-6.35" y="8.255" size="1.27" layer="25"/>
+<attribute name="VALUE" x="-6.35" y="0.635" size="1.27" layer="27"/>
+</element>
+<element name="U1" library="LinnesLab-Microcontrollers" package="ARTEMIS_CAST" value="" x="-21.59" y="3.81" smashed="yes">
+<attribute name="NAME" x="-21.59" y="24.13" size="1.27" layer="25"/>
+<attribute name="VALUE" x="-21.59" y="1.27" size="1.27" layer="27"/>
 </element>
 </elements>
@@
 <contactref element="USB1" pad="5"/>
 <contactref element="R4" pad="1"/>
-<wire x1="15.24" y1="19.05" x2="14" y2="12.935" width="0" layer="19" extent="1-1"/>
-<wire x1="14.39" y1="24.13" x2="15.24" y2="19.05" width="0" layer="19" extent="1-1"/>
-<wire x1="19.9" y1="24.13" x2="14.39" y2="24.13" width="0" layer="19" extent="1-1"/>
-<wire x1="23.71" y1="24.13" x2="19.9" y2="24.13" width="0" layer="19" extent="1-1"/>
-<wire x1="27.52" y1="24.13" x2="23.71" y2="24.13" width="0" layer="19" extent="1-1"/>
-<wire x1="31.33" y1="24.13" x2="27.52" y2="24.13" width="0" layer="19" extent="1-1"/>
+<contactref element="U$1" pad="1"/>
+<wire x1="27.52" y1="24.13" x2="31.33" y2="24.13" width="0" layer="19" extent="1-1"/>
+<wire x1="23.71" y1="24.13" x2="27.52" y2="24.13" width="0" layer="19" extent="1-1"/>
+<wire x1="19.9" y1="24.13" x2="23.71" y2="24.13" width="0" layer="19" extent="1-1"/>
 <wire x1="22.01" y1="27.94" x2="23.71" y2="24.13" width="0" layer="19" extent="1-1"/>
 <wire x1="22.86" y1="19.0199" x2="23.71" y2="24.13" width="0" layer="19" extent="1-1"/>
+<wire x1="14.39" y1="24.13" x2="19.9" y2="24.13" width="0" layer="19" extent="1-1"/>
+<wire x1="15.24" y1="19.05" x2="14.39" y2="24.13" width="0" layer="19" extent="1-1"/>
+<wire x1="14" y1="12.935" x2="15.24" y2="19.05" width="0" layer="19" extent="1-1"/>
+<wire x1="-6.35" y1="6.35" x2="14" y2="12.935" width="0" layer="19" extent="1-1"/>
 </signal>
 <signal name="VLIPO">
@@
 <wire x1="23.71" y1="27.94" x2="25.82" y2="27.94" width="0" layer="19" extent="1-1"/>
 </signal>
+<signal name="SDA">
+<contactref element="U$1" pad="4"/>
+</signal>
+<signal name="SCL">
+<contactref element="U$1" pad="3"/>
+</signal>
 </signals>
