File: Hardware/Top/SHY-TOP.brd (EAGLE design)
At the start: 160 x 100 mm, 0 parts

Commit message: Add top board
Parts:
- added C10, C11: 300p, LinnesLab-Passives:C0603
- added C12: 10u, LinnesLab-Passives:C0805
- added C13, C15, C17, C18, C19: 2.2uF, LinnesLab-Passives:C0402
- added C14: 100n, LinnesLab-Passives:C0603
- added C16: 10uF, LinnesLab-Passives:C0603
- added C2, C5, C6, C7: 1u, LinnesLab-Passives:C0603
- added C20, C21: 4.7u, LinnesLab-Passives:C0603
- added C8, C9: (no value), LinnesLab-Passives:C0603
- added CHRG2: MCP73831, LinnesLab-Power:SOT23-5
- added CORTEX1: CORTEX_DEBUG_PTH, LinnesLab-Connectors:2X5-PTH-1.27MM
- added D1, D4, D5: (no value), LinnesLab-DiscreteSemi:USC
- added J2: (no value), LinnesLab-Connectors:1X02
- added L2: 10u, LinnesLab-Passives:L0603
- added LDO2: MIC5504, LinnesLab-Power:SOT23-5
- added LED3: RED, LinnesLab-LED:LED-0603
- added LED4: BLUE, LinnesLab-LED:LED-0603
- added R11: (no value), LinnesLab-Passives:R0603
- added R12, R13, R14, R15: 100k, LinnesLab-Passives:R0603
- added R3, R4: 1k, LinnesLab-Passives:R0603
- added R5, R6, R8, R9: 10k, LinnesLab-Passives:R0603
- added R7: 390k, LinnesLab-Passives:R0603
- added SD2: (no value), LinnesLab-Connectors:MICROSD
- added SW1, SW6: SWITCH.MOM, LinnesLab-Switches:TACTILE_SWITCH_SMD_6.2MM_TALL
- added SW3, SW4: (no value), LinnesLab-Switches:BUTTON-GULLWING
- added U2: NRF52832_MODULE_MDBT42, LinnesLab-Microcontrollers:BLE_MODULE_RAYTAC_MDBT42
- added U3: (no value), LinnesLab-Displays:UG-2864HSWEG01_0.96IN_NO-WRAPAROUND
- added U4: PCF8523, LinnesLab-Clocks:SO8
- added USB2: USB.MICRO-BIGGERPADS, LinnesLab-Connectors:USB-MICRO-01.BIGGERPADS
- added XTAL2: 32.768kHz, LinnesLab-Clocks:2-SMD.NOLEAD.2.0MMTO1.2MM
- added XTAL3: 32.7680kHz, LinnesLab-Clocks:2-SMD.NOLEAD.2.0MMTO1.2MM
Connections:
- new net 3.3V: C12.2, C17.2, C19.2, C2.1, C6.1, CORTEX1.1, D1.-, LDO2.5, R15.2, R5.2, R8.2, R9.2, SD2.4, U2.11, U3.6, U3.9, U4.8
- new net BATT: R13.1, R14.2
- new net CD1: SD2.CD1
- new net CD2: SD2.CD2
- new net CHRG.STAT: CHRG2.1, R12.1
- new net CS.OLED: U3.13
- new net DC.OLED: U3.15
- new net DFU: SW3.3, U2.34
- new net DTR: C14.1
- new net FRST: U2.38
- new net GND: C10.2, C11.2, C12.1, C16.1, C17.1, C18.1, C19.1, C2.2, C20.2, C21.1, C5.1, C6.2, C7.2, C8.1, C9.2, CHRG2.2, CORTEX1.3, CORTEX1.5, CORTEX1.7, CORTEX1.9, J2.1, LDO2.2, LED3.C, LED4.C, R11.1, R14.1, R15.1, R6.1, R7.2, SD2.6, SD2.MT1, SD2.MT2, SW1.B1, SW1.B2, SW3.1, SW4.3, SW6.B1, SW6.B2, U2.1, U2.12, U2.24, U2.39, U3.1, U3.10, U3.12, U3.29, U3.30, U3.8, U4.4, USB2.5
- new net LED1: R3.2, U2.31
- new net LED2: R4.2, U2.33
- new net MISO: SD2.7, U2.28
- new net MOSI: SD2.3, U2.27, U3.19
- new net N$1: R6.2, U3.11
- new net N$10: LED4.A, R4.1
- new net N$11: L2.1, U2.10
- new net N$12: C7.1, L2.2, U2.9
- new net N$13: C16.2, U3.28
- new net N$14: CORTEX1.8
- new net N$15: C18.2, U3.27
- new net N$17: CHRG2.5, R11.2
- new net N$19: U4.2, XTAL3.P$1
- new net N$2: R7.1, U3.26
- new net N$20: U4.1, XTAL3.P$2
- new net N$3: C13.2, U3.2
- new net N$4: C8.2, U2.13, XTAL2.P$1
- new net N$5: C13.1, U3.3
- new net N$6: C9.1, U2.14, XTAL2.P$2
- new net N$7: C15.2, U3.4
- new net N$8: C15.1, U3.5
- new net N$9: LED3.A, R3.1
- new net P0.09/NFC1: C11.1, U2.22
- new net P0.10/NFC2: C10.1, U2.23
- new net RESET: C14.2, CORTEX1.10, D1.+, R5.1, SW4.1, U2.35
- new net RESET.OLED: U3.14
- new net RXD: U2.21
- new net SCK: SD2.5, U2.26, U3.18
- new net SCL: R8.1, U2.3, U4.6
- new net SD.CS: SD2.2
- new net SDA: R9.1, U2.2, U4.5
- new net SW1: SW1.A1, SW6.A1
- new net SWCLK: CORTEX1.4, U2.36
- new net SWDIO: CORTEX1.2, U2.37
- new net SWO: CORTEX1.6, U2.32
- new net TXD: U2.19
- new net USB+: USB2.3
- new net USB-: USB2.2
- new net VBAT: U4.3
- new net VIN: C21.2, C5.2, CHRG2.4, D4.-, D5.-, LDO2.1, LDO2.3, R12.2
- new net VLIPO: C20.1, CHRG2.3, D4.+, J2.2, R13.2
- new net V_USB: D5.+, USB2.1
Other:
- board size 160 x 100 mm -> 38 x 38 mm

Commit message: top board design
Parts:
- removed R8, R9: 10k, LinnesLab-Passives:R0603
- added C22: 100n, LinnesLab-Passives:C0603
- added C23, C24: 47p, LinnesLab-Passives:C0603
- added J1: (no value), LinnesLab-Connectors:1X07
- added JP2: (no value), LinnesLab-Switches:SMT-JUMPER_2_NO_SILK
- added LED5: RED, LinnesLab-LED:LED-0603
- added LED6: YELLOW, LinnesLab-LED:LED-0603
- added R1, R2: 10K, LinnesLab-Passives:R0603
- added R17, R18: 27, LinnesLab-Passives:R0603
- added R19, R20: 1k, LinnesLab-Passives:R0603
- added R21, R22: 0, LinnesLab-Passives:R0603
- added U5: FT231XS, LinnesLab-DigitalIC:SSOP20_L
- moved C18 4.11 mm to (29.0, 24.6)
- moved C16 3.79 mm to (30.3, 24.8)
Connections:
- net CHRG.STAT renamed D27/CHRG.STATUS
- removed net BATT: R13.1, R14.2
- removed net CD1: SD2.CD1
- removed net CS.OLED: U3.13
- removed net DC.OLED: U3.15
- removed net RESET.OLED: U3.14
- removed net RXD: U2.21
- removed net SD.CS: SD2.2
- removed net SW1: SW1.A1, SW6.A1
- removed net TXD: U2.19
- new net !CTS: JP2.2, U5.9
- new net !DTR: U5.1
- new net A4/BATT: R13.1, R14.2, U2.5
- new net A6/TIA: U2.7
- new net A7/PPG: U2.8
- new net D11/SW1: SW6.A1, U2.25
- new net D15/SW2: SW1.A1, U2.29
- new net D16/CS.OLED: U2.30, U3.13
- new net D27/CHRC.STATUS: U2.4
- new net D29/LED.CTRL: U2.6
- new net D3/RESET.OLED: U2.16, U3.14
- new net D4/DC.OLED: U2.17, U3.15
- new net D5/CD1: SD2.CD1, U2.18
- new net D7/SD.CS: SD2.2, U2.20
- new net FT3V3: U5.13
- new net N$16: R21.1
- new net N$23: R17.2, U5.12
- new net N$24: R18.2, U5.11
- new net N$25: LED5.C, R19.2
- new net N$26: LED6.C, R20.2
- new net RXD.FT: R22.1, U5.4
- new net RXD.NRF: R21.2, U2.21
- new net RXLED: R19.1, U5.17
- new net TXD.FT: U5.20
- new net TXD.NRF: R22.2, U2.19
- new net TXLED: R20.1, U5.10
- net 3.3V: now also C22.2, LED5.A, LED6.A, R1.2, R2.1, U5.14, U5.3; no longer R8.2, R9.2
- net GND: now also C22.1, C23.2, C24.1, JP2.1, U5.16, U5.6
- net SCL: now also R2.2; no longer R8.1
- net SDA: now also R1.1; no longer R9.1
- net USB+: now also C23.1, R18.1
- net USB-: now also C24.2, R17.1
- net V_USB: now also U5.15

Commit message: update D2/pin15 connection
Parts:
- added GPS.PWR: MIC5504, LinnesLab-Power:SOT23-5
Connections:
- new net D2/GPS.PWR: GPS.PWR.3, U2.15
Changed lines of the file:
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@@
 <attribute name="VALUE" x="3.73" y="30.968" size="0.6096" layer="27" font="vector" ratio="20"/>
+</element>
+<element name="GPS.PWR" library="LinnesLab-Power" package="SOT23-5" value="MIC5504" x="1.9304" y="-15.621" smashed="yes">
+<attribute name="NAME" x="0.0254" y="-15.621" size="0.6096" layer="25" ratio="20" rot="R90" align="bottom-center"/>
+<attribute name="VALUE" x="4.4704" y="-15.621" size="0.6096" layer="27" ratio="20" rot="R90" align="bottom-center"/>
 </element>
 </elements>
@@
 <wire x1="17.5174" y1="18.8914" x2="30.1468" y2="21.2552" width="0" layer="19" extent="1-1"/>
 </signal>
+<signal name="D2/GPS.PWR">
+<contactref element="U2" pad="15"/>
+<contactref element="GPS.PWR" pad="3"/>
+<wire x1="2.8804" y1="-16.9211" x2="29.4468" y2="21.2552" width="0" layer="19" extent="1-1"/>
+</signal>
 </signals>
